File: full_bridge_smps_kicad/EMI Filter and Rectification.kicad_sch (KiCad schematic)
At the start: 52 parts, among them J4 Conn_01x04_Male, J6 Conn_01x04_Male, J7 Conn_01x02_Male, J8 Conn_01x02_Male, Q1 IPW60R041C6, Q1 MMBT2904, Q2 IPW60R041C6, Q2 MMBT2904, Q3 IPW60R041C6, Q4 IPW60R041C6, SW1 SW_SPST, U2 UCC27323D

Commit message: Adding schematic
Other:
- note added: "*Separate PCB"
Changed lines of the file:
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@@
     (effects (font (size 4 4) (thickness 0.8) bold) (justify left bottom))
+  )
+  (text "*Separate PCB" (at 60.96 104.14 0)
+    (effects (font (size 1.27 1.27)) (justify left bottom))
+  )
+  (text "*Separate PCB" (at 143.51 105.41 0)
+    (effects (font (size 1.27 1.27)) (justify left bottom))
   )
   (text "AUXILIARY RECTIFICATION\n" (at 205.74 29.21 0)
