File: full_bridge_smps_kicad/Full Bridge Current Feedback and Drive.kicad_sch (KiCad schematic)
At the start: 27 parts, among them U10 UCC27324D, U19 UCC27324D, U8 OPA333AID

Commit message: A bit of refactoring, saving work for the day
Parts:
- removed C18 (x3): 100nF, symbol Device:C
- removed R53 (x3): 2.21k, symbol Device:R_US
- removed R53 (x2): 10.0, symbol Device:R_US
- added C18: 1uF, symbol Device:C
- added C18 (x2): 100nF, symbol Device:C
- added R53 (x2): 10.0, symbol Device:R_US
- added R53 (x2): 1.00k, symbol Device:R_US
Connections:
- net +3V45: now also R53.1
- net GNDREF: now also C18.1, C18.1, R53.2
- net OUT_CURR: now also C18.2, R53.2
- net V+: now also C18.2, R53.2
- net at U8.2 (IN-): now also C18.1, R53.1, R53.1
- net at U8.3 (IN+): now also C18.2, R53.2
Other:
- note added: "OUTPUT CURRENT MEASUREMENT"
- note added: "PRIMARY CURRENT FEEDBACK"
- moved on the sheet: C18, D18B, D19B, D20A, D20B, D23A, D5, U10A, U10B, U10C, U19A, U19B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
