File: full_bridge_smps_kicad/PFC Feedback and Control.kicad_sch (KiCad schematic)
At the start: 57 parts, among them J8 Conn_01x06_Male, J9 Conn_01x06_Male, U7 UCC28070PW

Commit message: A bit of refactoring, saving work for the day
Other:
- moved on the sheet: SC2
Changed lines of the file:
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@@
     (stroke (width 0) (type default))
   )
-  (wire (pts (xy 228.6 99.06) (xy 231.14 99.06))
+  (wire (pts (xy 236.22 106.68) (xy 238.76 106.68))
     (stroke (width 0) (type default))
   )
@@
     (stroke (width 0) (type default))
   )
-  (wire (pts (xy 238.76 99.06) (xy 241.3 99.06))
+  (wire (pts (xy 246.38 106.68) (xy 248.92 106.68))
     (stroke (width 0) (type default))
   )
@@
     )
   )
-  (symbol (lib_id "Device:R_US") (at 234.95 99.06 90) (unit 1)
-    (in_bom yes) (on_board yes) (dnp no)
-    (property "Reference" "SC2" (at 233.68 96.52 90)
-      (effects (font (size 1.27 1.27)))
-    )
-    (property "Value" "0" (at 234.95 101.6 90)
-      (effects (font (size 1.27 1.27)))
-    )
-    (property "Footprint" "" (at 235.204 98.044 90)
-      (effects (font (size 1.27 1.27)) hide)
-    )
-    (property "Datasheet" "~" (at 234.95 99.06 0)
+  (symbol (lib_id "Device:R_US") (at 242.57 106.68 90) (unit 1)
+    (in_bom yes) (on_board yes) (dnp no)
+    (property "Reference" "SC2" (at 241.3 104.14 90)
+      (effects (font (size 1.27 1.27)))
+    )
+    (property "Value" "0" (at 242.57 109.22 90)
+      (effects (font (size 1.27 1.27)))
+    )
+    (property "Footprint" "" (at 242.824 105.664 90)
+      (effects (font (size 1.27 1.27)) hide)
+    )
+    (property "Datasheet" "~" (at 242.57 106.68 0)
       (effects (font (size 1.27 1.27)) hide)
     )
@@
     )
   )
-  (symbol (lib_id "power:GNDPWR") (at 241.3 99.06 0) (unit 1)
+  (symbol (lib_id "power:GNDPWR") (at 248.92 106.68 0) (unit 1)
     (in_bom yes) (on_board yes) (dnp no) (fields_autoplaced)
-    (property "Reference" "#PWR047" (at 241.3 104.14 0)
-      (effects (font (size 1.27 1.27)) hide)
-    )
-    (property "Value" "GNDPWR" (at 241.173 102.87 0)
-      (effects (font (size 1.27 1.27)))
-    )
-    (property "Footprint" "" (at 241.3 100.33 0)
-      (effects (font (size 1.27 1.27)) hide)
-    )
-    (property "Datasheet" "" (at 241.3 100.33 0)
+    (property "Reference" "#PWR047" (at 248.92 111.76 0)
+      (effects (font (size 1.27 1.27)) hide)
+    )
+    (property "Value" "GNDPWR" (at 248.793 110.49 0)
+      (effects (font (size 1.27 1.27)))
+    )
+    (property "Footprint" "" (at 248.92 107.95 0)
+      (effects (font (size 1.27 1.27)) hide)
+    )
+    (property "Datasheet" "" (at 248.92 107.95 0)
       (effects (font (size 1.27 1.27)) hide)
     )
@@
     )
   )
-  (symbol (lib_id "power:GND1") (at 228.6 99.06 0) (unit 1)
-    (in_bom yes) (on_board yes) (dnp no)
-    (property "Reference" "#PWR057" (at 228.6 105.41 0)
-      (effects (font (size 1.27 1.27)) hide)
-    )
-    (property "Value" "GND1" (at 228.6 102.87 0)
-      (effects (font (size 1.27 1.27)))
-    )
-    (property "Footprint" "" (at 228.6 99.06 0)
-      (effects (font (size 1.27 1.27)) hide)
-    )
-    (property "Datasheet" "" (at 228.6 99.06 0)
-      (effects (font (size 1.27 1.27)) hide)
-    )
+  (symbol (lib_id "power:GND1") (at 236.22 106.68 0) (unit 1)
+    (in_bom yes) (on_board yes) (dnp no)
+    (property "Reference" "#PWR057" (at 236.22 113.03 0)
+      (effects (font (size 1.27 1.27)) hide)
+    )
+    (property "Value" "GND1" (at 236.22 110.49 0)
+      (effects (font (size 1.27 1.27)))
+    )
+    (property "Footprint" "" (at 236.22 106.68 0)
+      (effects (font (size 1.27 1.27)) hide)
+    )
+    (property "Datasheet" "" (at 236.22 106.68 0)
+      (effects (font (size 1.27 1.27)) hide)
+    )
