File: full_bridge_smps_kicad/Secondary Rectification.kicad_sch (KiCad schematic)
At the start: 45 parts, among them Q16 IPB081N06L3 G, Q17 IPB081N06L3 G, Q18 IPB081N06L3 G, Q8 IPB081N06L3 G, U11 UCC27324D, U12 UCC27324D, U5 UCC27324D

Commit message: A bit of refactoring, saving work for the day
Parts:
- added C18 (x2): DNP, symbol Device:C
- added C18 (x3): 10uF, symbol Device:C
- added C18 (x2): 100nF, symbol Device:C
- added D31: LED, symbol Device:LED
- added L3 (x4): 50nH, symbol Device:L
- added L9: 10uH, symbol Device:L_Coupled
- added R53: 4.32k, symbol Device:R_US
- added R53: 0.2m, symbol Device:R_US
Connections:
- net GNDREF: now also C18.1, C18.2, R53.1
- net VOUT: now also L9.1
- new net: L3.1, L3.2, L9.4
- new net: D31.2 (A), R53.2
- new net: L3.1, L3.2, L9.2
- new net OUTPUT+: C18.2, C18.2, C18.2, C18.2, C18.2, C18.2, L3.1, L3.2, R53.1
- new net OUTPUT-: C18.1, C18.1, C18.1, C18.1, C18.1, C18.1, D31.1 (K), L3.1, L3.2
- new net OUT_CURR_SEN: L9.3, R53.2
Other:
- note added: "One turn per side"
- note added: "Phase 1"
- note added: "Phase 2"
- moved on the sheet: C18, C68, C72, C78, D5, L3, Q16, Q17, Q18, Q8, R53, U11A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
